Commit message: robot

File: body.urdf (robot description, URDF)
Before this commit: robot robot, 2 links, 1 joints
Links:
- removed link Leg
- added link BackLeg, mass 1; collision box size=1 1 1; visual box size=1 1 1
- added link FrontLeg, mass 1; collision box size=1 1 1; visual box size=1 1 1
Joints:
- removed joint Torso_Leg
- added joint FrontLeg_Torso: type revolute, parent FrontLeg, child Torso, origin xyz=1 0 1 rpy=0 0 0, axis 0 1 0, limit lower=-3.14159 upper=3.14159 effort=0.0 velocity=0.0
- added joint Torso_BackLeg: type revolute, parent Torso, child BackLeg, origin xyz=1 0 0 rpy=0 0 0, axis 0 1 0, limit lower=-3.14159 upper=3.14159 effort=0.0 velocity=0.0

Commit message: joints

File: body.urdf (robot description, URDF)
Before this commit: robot robot, 3 links, 2 joints
Links:
- removed link BackLeg
- removed link FrontLeg
- removed link Torso
- added link backleg, mass 1; collision box size=1 1 1; visual box size=1 1 1
- added link frontleg, mass 1; collision box size=1 1 1; visual box size=1 1 1
- added link torso, mass 1; collision box size=1 1 1; visual box size=1 1 1
Joints:
- removed joint FrontLeg_Torso
- removed joint Torso_BackLeg
- added joint frontleg_torso: type revolute, parent frontleg, child torso, origin xyz=1 0 1 rpy=0 0 0, axis 0 1 0, limit lower=-3.14159 upper=3.14159 effort=0.0 velocity=0.0
- added joint torso_backleg: type revolute, parent torso, child backleg, origin xyz=1 0 0 rpy=0 0 0, axis 0 1 0, limit lower=-3.14159 upper=3.14159 effort=0.0 velocity=0.0

Commit message: motors

File: body.urdf (robot description, URDF)
Before this commit: robot robot, 3 links, 2 joints
Joints:
- removed joint frontleg_torso
- added joint torso_frontleg: type revolute, parent frontleg, child torso, origin xyz=1 0 1 rpy=0 0 0, axis 0 1 0, limit lower=-3.14159 upper=3.14159 effort=0.0 velocity=0.0

Commit message: first commit to refactoring

File: body.urdf (robot description, URDF)
Before this commit: robot robot, 3 links, 2 joints
Joints:
- joint torso_backleg: origin xyz=1 0 0 rpy=0 0 0 -> xyz=2 0 1 rpy=0 0 0
- joint torso_frontleg: child torso -> frontleg; parent frontleg -> torso

Commit message: saving

File: body.urdf (robot description, URDF)
Before this commit: robot robot, 3 links, 2 joints
Links:
- link backleg: geometry collision box size=0.2 1 0.2; visual box size=0.2 1 0.2
- link frontleg: geometry collision box size=0.2 1 0.2; visual box size=0.2 1 0.2
Joints:
- joint torso_backleg: origin xyz=2 0 1 rpy=0 0 0 -> xyz=0 -0.5 1 rpy=0 0 0
- joint torso_frontleg: origin xyz=1 0 1 rpy=0 0 0 -> xyz=0 0.5 1 rpy=0 0 0

Commit message: quadruped

File: body.urdf (robot description, URDF)
Before this commit: robot robot, 3 links, 2 joints
Links:
- added link backleg2, mass 1; collision box size=0.2 0.2 1; visual box size=0.2 0.2 1
- added link frontleg2, mass 1; collision box size=0.2 0.2 1; visual box size=0.2 0.2 1
- added link leftleg, mass 1; collision box size=1 0.2 0.2; visual box size=1 0.2 0.2
- added link leftleg2, mass 1; collision box size=0.2 0.2 1; visual box size=0.2 0.2 1
- added link rightleg, mass 1; collision box size=1 0.2 0.2; visual box size=1 0.2 0.2
- added link rightleg2, mass 1; collision box size=0.2 0.2 1; visual box size=0.2 0.2 1
Joints:
- added joint backleg_backleg2: type revolute, parent backleg, child backleg2, origin xyz=0 -1 0 rpy=0 0 0, axis 1 0 0, limit lower=-3.14159 upper=3.14159 effort=0.0 velocity=0.0
- added joint frontleg_frontleg2: type revolute, parent frontleg, child frontleg2, origin xyz=0 1 0 rpy=0 0 0, axis 1 0 0, limit lower=-3.14159 upper=3.14159 effort=0.0 velocity=0.0
- added joint leftleg_leftleg2: type revolute, parent leftleg, child leftleg2, origin xyz=-1 0 0 rpy=0 0 0, axis 0 1 0, limit lower=-3.14159 upper=3.14159 effort=0.0 velocity=0.0
- added joint rightleg_rightleg2: type revolute, parent rightleg, child rightleg2, origin xyz=1 0 0 rpy=0 0 0, axis 0 1 0, limit lower=-3.14159 upper=3.14159 effort=0.0 velocity=0.0
- added joint torso_leftleg: type revolute, parent torso, child leftleg, origin xyz=-0.5 0 1 rpy=0 0 0, axis 0 1 0, limit lower=-3.14159 upper=3.14159 effort=0.0 velocity=0.0
- added joint torso_rightleg: type revolute, parent torso, child rightleg, origin xyz=0.5 0 1 rpy=0 0 0, axis 0 1 0, limit lower=-3.14159 upper=3.14159 effort=0.0 velocity=0.0
- joint torso_backleg: axis 0 1 0 -> 1 0 0
- joint torso_frontleg: axis 0 1 0 -> 1 0 0

Commit message: housekeeping:

File: body.urdf (robot description, URDF)
Before this commit: robot robot, 9 links, 8 joints
Links:
- link torso: geometry collision box size=1 1 4; visual box size=1 1 4

Commit message: housekeeping

File: body.urdf (robot description, URDF)
Before this commit: robot robot, 9 links, 8 joints
Links:
- link torso: geometry collision box size=1 1 1; visual box size=1 1 1

Commit message: finished new designs

File: body.urdf (robot description, URDF)
Before this commit: robot robot, 9 links, 8 joints
Links:
- link backleg: geometry collision box size=1 0.2 0.2; visual box size=1 0.2 0.2
- link frontleg: geometry collision box size=1 0.2 0.2; visual box size=1 0.2 0.2
- link torso: geometry collision box size=1 3 1; visual box size=1 3 1
Joints:
- joint backleg_backleg2: axis 1 0 0 -> 0 1 0; origin xyz=0 -1 0 rpy=0 0 0 -> xyz=-1 -0.5 0 rpy=0 0 0
- joint frontleg_frontleg2: axis 1 0 0 -> 0 1 0; origin xyz=0 1 0 rpy=0 0 0 -> xyz=1 -0.5 0 rpy=0 0 0
- joint leftleg_leftleg2: origin xyz=-1 0 0 rpy=0 0 0 -> xyz=-1 0.5 0 rpy=0 0 0
- joint rightleg_rightleg2: origin xyz=1 0 0 rpy=0 0 0 -> xyz=1 0.5 0 rpy=0 0 0
- joint torso_backleg: axis 1 0 0 -> 0 1 0; origin xyz=0 -0.5 1 rpy=0 0 0 -> xyz=-0.5 -0.5 1 rpy=0 0 0
- joint torso_frontleg: axis 1 0 0 -> 0 1 0; origin xyz=0 0.5 1 rpy=0 0 0 -> xyz=0.5 -0.5 1 rpy=0 0 0
- joint torso_leftleg: origin xyz=-0.5 0 1 rpy=0 0 0 -> xyz=-0.5 0.5 1 rpy=0 0 0
- joint torso_rightleg: origin xyz=0.5 0 1 rpy=0 0 0 -> xyz=0.5 0.5 1 rpy=0 0 0

Commit message: edits

File: body.urdf (robot description, URDF)
Before this commit: robot robot, 9 links, 8 joints
Links:
- removed link backleg
- removed link backleg2
- removed link frontleg
- removed link frontleg2
- removed link leftleg
- removed link leftleg2
- removed link rightleg
- removed link rightleg2
- removed link torso
- added link 0, mass 1; collision box size=1.23 1.77 0.73; visual box size=1.23 1.77 0.73
- added link 1, mass 1; collision box size=1.18 0.84 1.73; visual box size=1.18 0.84 1.73
- added link 2, mass 1; collision box size=1.61 0.92 1.36; visual box size=1.61 0.92 1.36
- added link 3, mass 1; collision box size=0.68 0.94 1.66; visual box size=0.68 0.94 1.66
Joints:
- removed joint backleg_backleg2
- removed joint frontleg_frontleg2
- removed joint leftleg_leftleg2
- removed joint rightleg_rightleg2
- removed joint torso_backleg
- removed joint torso_frontleg
- removed joint torso_leftleg
- removed joint torso_rightleg
- added joint 0_1: type revolute, parent 0, child 1, origin xyz=0 1.77 0.365 rpy=0 0 0, axis 0 0 1, limit lower=-3.14159 upper=3.14159 effort=0.0 velocity=0.0
- added joint 1_2: type revolute, parent 1, child 2, origin xyz=0 0.84 0.31500000000000006 rpy=0 0 0, axis 0 0 1, limit lower=-3.14159 upper=3.14159 effort=0.0 velocity=0.0
- added joint 2_3: type revolute, parent 2, child 3, origin xyz=0 0.92 0.0 rpy=0 0 0, axis 0 0 1, limit lower=-3.14159 upper=3.14159 effort=0.0 velocity=0.0
